File: JanusV1.sch (EAGLE design)
At the start: 0 parts

Commit message: Version1.0.0
The schematic is ready to go with the exception of unspecified
connectors. Will update when connectors are specified.
Parts:
- added C1: 100nF, resistor:C-EUC0603
- added C2: .01uF, resistor:C-EUC0603
- added D1: 1N4148X-TP, CP-Discrete:1N4148X-TP
- added OK1, OK2, OK3: TLP152, CP-Discrete:TLP152
- added Q1, Q2: DMN6140L-7, CP-Discrete:DMN6140L-7
- added R1, R2, R3, R4: 1M, resistor:R-US_R0603
- added U1: SN74LV08APWR, CP-IC:SN74LV08APWR
- added U2: 74LVC1G86W5-7, CP-IC:74LVC1G86W5-7
- added U3: NE555S-13DICT-ND, CP-IC:NE555S-13DICT-ND
- added U4: 74HCT1G14GW,125, CP-IC:74HCT1G14GW,125
Connections:
- new net +5V: OK1.P$6, OK2.P$6, OK3.P$6, U1.P$14, U2.P$5, U4.P$5
- new net AUTO: U1.P$2
- new net COMPDRIVE: OK3.P$1, U1.P$3, U1.P$4
- new net COMPDRIVE_ISO: OK3.P$5
- new net COMPDRIVE_R: OK3.P$2, R4.1
- new net DELAYED: U1.P$10, U1.P$13, U3.OUT
- new net ENABLE: C1.1, U1.P$6, U3.RES, U3.VCC
- new net FOR: OK1.P$5, U1.P$12, U2.P$1
- new net FORSOL: Q2.D
- new net FOR_CTRL: Q2.G, U1.P$11
- new net FOR_ISO: OK1.P$1
- new net FOR_ISO_R: OK1.P$2, OK2.P$2, R2.2, R3.2
- new net GND: C2.2, D1.P$1, OK1.P$4, OK2.P$4, OK3.P$4, Q1.S, Q2.S, R1.1, R2.1, R3.1, R4.2, U1.P$7, U2.P$3, U3.GND, U4.P$3
- new net N$5: U1.P$5, U2.P$4
- new net N$6: C2.1, U3.CONT
- new net NEUTRAL: U4.P$2
- new net N_NEUTRAL: U1.P$1, U4.P$4
- new net REV: OK2.P$5, U1.P$9, U2.P$2
- new net REVSOL: Q1.D
- new net REV_CTRL: Q1.G, U1.P$8
- new net REV_ISO: OK2.P$1
- new net THRESTRIG: C1.2, D1.P$2, R1.2, U3.THRE, U3.TRIG
